File: hardware/footswitch/anthracite-footswitch.kicad_pcb (KiCad board)
At the start: 2 copper layers, 14 x 16.1 mm, 2 parts, among them J1 Conn_01x03_Socket, SW1 SW_DPDT_x2

Commit message: Mark the footswitch board with v1.0 on the silkscreen
The top and bottom boards already carry "V1.0 CERN-OHL-S-2.0" and the source
URL; the footswitch board is 14 x 16 mm, so it carries the version only.
Board STEP and schematic PDF re-exported.

Co-Authored-By: Claude Opus 5 <noreply@anthropic.com>
Claude-Session: https://claude.ai/code/session_01H9QGzk7saaLy5LAwVYL6Ej
Other:
- board text added: "v1.0"
Changed lines of the file:
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@@
 		(layer "Edge.Cuts")
+	)
+	(gr_text "v1.0"
+		(at 40 24.1 0)
+		(layer "B.SilkS")
+		(effects
+			(font
+				(size 1.2 1.2)
+			)
+			(justify left top mirror)
+		)
 	)
 	(segment
